File: pcb/esphome-humitemp.kicad_sch (KiCad schematic)
At the start: 17 parts, among them J2 USB_IN, SW1 RESET, U1 SHT3x, U3 AMS1117-3.3, U4 ESP32-C3-MINI-1

Commit message: v3
Parts:
- removed H1, H2: MountingHole, MountingHole:MountingHole_3.2mm_M3, symbol Mechanical:MountingHole
- removed U3: AMS1117-3.3, Package_TO_SOT_SMD:SOT-223-3_TabPin2, symbol Regulator_Linear:AP1117-33
- added C6: 0.1u, Capacitor_SMD:C_0603_1608Metric, symbol Device:C_Small
- added U1: TLV75533PDRV, Package_SON:WSON-6-1EP_2x2mm_P0.65mm_EP1x1.6mm, symbol Regulator_Linear:TLV75533PDRV
- added U2: USBLC6-4SC6, Package_TO_SOT_SMD:SOT-23-6, symbol Power_Protection:USBLC6-4SC6
- J1: renamed from J2; footprint esphome-humitemp:MOLEX_48037-0001 -> Project specific:SHOU_HAN_AM90
- R11, R7: footprint Resistor_SMD:R_0402_1005Metric -> Resistor_SMD:R_0805_2012Metric
- R4: renamed from R3; footprint Resistor_SMD:R_0402_1005Metric -> Resistor_SMD:R_0805_2012Metric
- R5: renamed from R2; footprint Resistor_SMD:R_0402_1005Metric -> Resistor_SMD:R_0805_2012Metric
- renumbered C1 to C3, C5 to C4, C2 to C5, U4 to U3, U1 to U4
Connections:
- net +3V3: now also C6.2, U1.1 (OUT)
- net D+: now also U2.3 (I/O2), U2.4 (I/O3)
- net D-: now also U2.1 (I/O1), U2.6 (I/O4)
- net GND: now also C6.1, U1.3 (GND), U1.7 (GND), U2.2 (GND)
- net VBUS: now also U1.4 (EN), U1.6 (IN), U2.5 (VBUS)
Other:
- note removed: "Mechanical"
- moved on the sheet: R4, R5, U4

Commit message: Ready for final checking
Parts:
- removed C1: 10u, Capacitor_SMD:C_0805_2012Metric, symbol Device:C_Small
- removed U1: TLV75533PDRV, Package_SON:WSON-6-1EP_2x2mm_P0.65mm_EP1x1.6mm, symbol Regulator_Linear:TLV75533PDRV
- added U1: TLV75533PDBV, Package_TO_SOT_SMD:SOT-23-5, symbol Regulator_Linear:TLV75533PDBV
- C1: value 10u -> 1u; footprint Capacitor_SMD:C_0805_2012Metric -> Capacitor_SMD:C_0603_1608Metric
- C3, C5: value 1uF -> 10uF; footprint Capacitor_SMD:C_0805_2012Metric -> Capacitor_SMD:C_0603_1608Metric; LCSC C28323 -> C19702
- R11, R4, R5, R7: footprint Resistor_SMD:R_0805_2012Metric -> Resistor_SMD:R_0402_1005Metric
- SW1: footprint Button_Switch_SMD:SW_Push_1P1T_XKB_TS-1187A -> EasyEda:SW-SMD_L3.0-W2.5-P3.40-LS4.0-EH
Connections:
- net +3V3: now also U1.5 (OUT)
- net GND: now also U1.2 (GND)
- net VBUS: now also U1.1 (IN), U1.3 (EN)
- net GPIO0: no longer names the net of SW1.1 (A), U3.23 (GPIO9)
Other:
- note removed: "C3 uses GPIO9 now"
- moved on the sheet: C4
